File: STLink_V3E_Module.kicad_sch (KiCad schematic)
At the start: 47 parts

Commit message: kicad xfer
Parts:
- C26, C34, C41, C42, C63, C90, CN1, CN16, CN2, HW1, HW11, HW12, HW13, HW14, HW15, HW16, JP6, JP8, LED4, LED6, R1, R10, R11, R12, R13, R14, R15, R16, R17, R18, R19, R20, R25, R3, R4, R6, R7, R8, R9, U10, U15, U16, U17, U18, U5, U9, X1: value ~ -> (none)
Changed lines of the file:
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@@
 			)
 		)
-		(property "Value" "~"
+		(property "Value" ""
 			(at 264.16 24.5872 0)
 			(effects
@@
 			)
 		)
-		(property "Value" "~"
+		(property "Value" ""
 			(at 35.56 133.8072 0)
 			(effects
@@
 			)
 		)
-		(property "Value" "~"
+		(property "Value" ""
 			(at 279.4 24.5872 0)
 			(effects
@@
 			)
 		)
-		(property "Value" "~"
+		(property "Value" ""
 			(at 37.592 45.1612 0)
 			(effects
@@
 			)
 		)
-		(property "Value" "~"
+		(property "Value" ""
 			(at 165.1 98.2472 0)
 			(effects
@@
 			)
 		)
-		(property "Value" "~"
+		(property "Value" ""
 			(at 38.1 187.1472 0)
 			(effects
@@
 			)
 		)
-		(property "Value" "~"
+		(property "Value" ""
 			(at 212.852 160.9852 0)
 			(effects
@@
 			)
 		)
-		(property "Value" "~"
+		(property "Value" ""
 			(at 277.114 95.1992 0)
 			(effects
@@
 			)
 		)
-		(property "Value" "~"
+		(property "Value" ""
 			(at 220.98 49.9872 0)
 			(effects
@@
 			)
 		)
-		(property "Value" "~"
+		(property "Value" ""
 			(at 220.98 42.3672 0)
 			(effects
@@
 			)
 		)
-		(property "Value" "~"
+		(property "Value" ""
 			(at 46.736 173.9392 0)
 			(effects
@@
 			)
 		)
-		(property "Value" "~"
+		(property "Value" ""
 			(at 91.44 199.8472 0)
 			(effects
@@
 			)
 		)
-		(property "Value" "~"
+		(property "Value" ""
 			(at 248.92 49.9872 0)
 			(effects
@@
 			)
 		)
-		(property "Value" "~"
+		(property "Value" ""
 			(at 204.978 92.6592 0)
 			(effects
@@
 			)
 		)
-		(property "Value" "~"
+		(property "Value" ""
 			(at 271.78 24.5872 0)
 			(effects
@@
 			)
 		)
-		(property "Value" "~"
+		(property "Value" ""
 			(at 7.874 158.6992 0)
 			(effects
@@
 			)
 		)
-		(property "Value" "~"
+		(property "Value" ""
 			(at 165.1 105.8672 0)
 			(effects
@@
 			)
 		)
-		(property "Value" "~"
+		(property "Value" ""
 			(at 220.98 47.4472 0)
 			(effects
@@
 			)
 		)
-		(property "Value" "~"
+		(property "Value" ""
 			(at 256.54 24.5872 0)
 			(effects
@@
 			)
 		)
-		(property "Value" "~"
+		(property "Value" ""
 			(at 7.62 34.7472 0)
 			(effects
@@
 			)
 		)
-		(property "Value" "~"
+		(property "Value" ""
 			(at 220.98 37.2872 0)
 			(effects
@@
 			)
 		)
-		(property "Value" "~"
+		(property "Value" ""
 			(at 25.4 164.2872 0)
 			(effects
@@
 			)
 		)
-		(property "Value" "~"
+		(property "Value" ""
 			(at 139.192 90.6272 0)
 			(effects
@@
 			)
 		)
-		(property "Value" "~"
+		(property "Value" ""
 			(at 240.538 97.7392 0)
 			(effects
@@
 			)
 		)
-		(property "Value" "~"
+		(property "Value" ""
 			(at 157.48 44.9072 0)
 			(effects
@@
 			)
 		)
-		(property "Value" "~"
+		(property "Value" ""
 			(at 212.852 166.0652 0)
 			(effects
@@
 			)
 		)
-		(property "Value" "~"
+		(property "Value" ""
 			(at 71.374 184.0992 0)
 			(effects
@@
 			)
 		)
-		(property "Value" "~"
+		(property "Value" ""
 			(at 157.48 49.9872 0)
 			(effects
@@
 			)
 		)
-		(property "Value" "~"
+		(property "Value" ""
 			(at 12.7 105.8672 0)
 			(effects
@@
 			)
 		)
-		(property "Value" "~"
+		(property "Value" ""
 			(at 68.072 34.7472 0)
 			(effects
@@
 			)
 		)
-		(property "Value" "~"
+		(property "Value" ""
 			(at 248.92 88.0872 0)
 			(effects
@@
 			)
 		)
-		(property "Value" "~"
+		(property "Value" ""
 			(at 212.852 163.5252 0)
 			(effects
@@
 			)
 		)
-		(property "Value" "~"
+		(property "Value" ""
 			(at 58.42 154.1272 0)
 			(effects
@@
 			)
 		)
-		(property "Value" "~"
+		(property "Value" ""
 			(at 182.88 55.0672 0)
 			(effects
@@
 			)
 		)
-		(property "Value" "~"
+		(property "Value" ""
 			(at 203.2 102.8192 0)
 			(effects
@@
 			)
 		)
-		(property "Value" "~"
+		(property "Value" ""
 			(at 83.058 186.6392 0)
 			(effects
@@
 			)
 		)
-		(property "Value" "~"
+		(property "Value" ""
 			(at 241.3 24.5872 0)
 			(effects
@@
 			)
 		)
-		(property "Value" "~"
+		(property "Value" ""
 			(at 248.92 24.5872 0)
 			(effects
@@
 			)
 		)
-		(property "Value" "~"
+		(property "Value" ""
 			(at 215.138 92.6592 0)
 			(effects
@@
 			)
 		)
-		(property "Value" "~"
+		(property "Value" ""
 			(at 220.98 39.8272 0)
 			(effects
@@
 			)
 		)
-		(property "Value" "~"
+		(property "Value" ""
 			(at 48.26 49.4792 0)
 			(effects
@@
 			)
 		)
-		(property "Value" "~"
+		(property "Value" ""
 			(at 53.594 173.9392 0)
 			(effects
@@
 			)
 		)
-		(property "Value" "~"
+		(property "Value" ""
 			(at 93.472 88.0872 0)
 			(effects
@@
 			)
 		)
-		(property "Value" "~"
+		(property "Value" ""
 			(at 212.852 168.6052 0)
 			(effects
@@
 			)
 		)
-		(property "Value" "~"
+		(property "Value" ""
 			(at 17.78 159.2072 0)
 			(effects
@@
 			)
 		)
-		(property "Value" "~"
+		(property "Value" ""
 			(at 47.752 88.0872 0)
 			(effects
@@
 			)
 		)
-		(property "Value" "~"
+		(property "Value" ""
 			(at 193.294 95.1992 0)
 			(effects
