File: STLink_V3E_PWR.kicad_sch (KiCad schematic)
At the start: 65 parts

Commit message: kicad xfer
Parts:
- C10, C100, C101, C18, C23, C28, C29, C32, C33, C36, C39, C40, C45, C46, C47, C48, C49, C50, C51, C52, C53, C54, C55, C56, C57, C58, C59, C60, C61, C62, C64, C65, C66, C9, C98, C99, CN11, CN4, D1, D2, D3, HW21, HW4, HW5, HW6, HW7, HW8, HW9, JP1, JP2, JP4, JP5, JP7, JP9, LED5, R24, R5, SB1, SB27, SB28, SB32, U2, U7, U8, U9: value ~ -> (none)
Changed lines of the file:
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@@
 			)
 		)
-		(property "Value" "~"
+		(property "Value" ""
 			(at 239.014 46.9392 0)
 			(effects
@@
 			)
 		)
-		(property "Value" "~"
+		(property "Value" ""
 			(at 210.82 100.7872 0)
 			(effects
@@
 			)
 		)
-		(property "Value" "~"
+		(property "Value" ""
 			(at 28.194 179.0192 0)
 			(effects
@@
 			)
 		)
-		(property "Value" "~"
+		(property "Value" ""
 			(at 78.994 156.1592 0)
 			(effects
@@
 			)
 		)
-		(property "Value" "~"
+		(property "Value" ""
 			(at 211.074 46.9392 0)
 			(effects
@@
 			)
 		)
-		(property "Value" "~"
+		(property "Value" ""
 			(at 113.792 67.5132 0)
 			(effects
@@
 			)
 		)
-		(property "Value" "~"
+		(property "Value" ""
 			(at 241.3 83.0072 0)
 			(effects
@@
 			)
 		)
-		(property "Value" "~"
+		(property "Value" ""
 			(at 213.36 83.0072 0)
 			(effects
@@
 			)
 		)
-		(property "Value" "~"
+		(property "Value" ""
 			(at 122.174 135.8392 0)
 			(effects
@@
 			)
 		)
-		(property "Value" "~"
+		(property "Value" ""
 			(at 68.834 133.2992 0)
 			(effects
@@
 			)
 		)
-		(property "Value" "~"
+		(property "Value" ""
 			(at 187.452 34.4932 0)
 			(effects
@@
 			)
 		)
-		(property "Value" "~"
+		(property "Value" ""
 			(at 132.334 135.8392 0)
 			(effects
@@
 			)
 		)
-		(property "Value" "~"
+		(property "Value" ""
 			(at 221.234 46.9392 0)
 			(effects
@@
 			)
 		)
-		(property "Value" "~"
+		(property "Value" ""
 			(at 254 121.1072 0)
 			(effects
@@
 			)
 		)
-		(property "Value" "~"
+		(property "Value" ""
 			(at 18.034 156.1592 0)
 			(effects
@@
 			)
 		)
-		(property "Value" "~"
+		(property "Value" ""
 			(at 259.334 46.9392 0)
 			(effects
@@
 			)
 		)
-		(property "Value" "~"
+		(property "Value" ""
 			(at 149.86 184.6072 0)
 			(effects
@@
 			)
 		)
-		(property "Value" "~"
+		(property "Value" ""
 			(at 58.674 133.2992 0)
 			(effects
@@
 			)
 		)
-		(property "Value" "~"
+		(property "Value" ""
 			(at 38.354 156.1592 0)
 			(effects
@@
 			)
 		)
-		(property "Value" "~"
+		(property "Value" ""
 			(at 18.034 133.2992 0)
 			(effects
@@
 			)
 		)
-		(property "Value" "~"
+		(property "Value" ""
 			(at 18.034 179.0192 0)
 			(effects
@@
 			)
 		)
-		(property "Value" "~"
+		(property "Value" ""
 			(at 19.558 90.1192 0)
 			(effects
@@
 			)
 		)
-		(property "Value" "~"
+		(property "Value" ""
 			(at 189.992 132.2832 0)
 			(effects
@@
 			)
 		)
-		(property "Value" "~"
+		(property "Value" ""
 			(at 213.36 128.7272 0)
 			(effects
@@
 			)
 		)
-		(property "Value" "~"
+		(property "Value" ""
 			(at 28.194 133.2992 0)
 			(effects
@@
 			)
 		)
-		(property "Value" "~"
+		(property "Value" ""
 			(at 193.04 184.6072 0)
 			(effects
@@
 			)
 		)
-		(property "Value" "~"
+		(property "Value" ""
 			(at 112.014 135.8392 0)
 			(effects
@@
 			)
 		)
-		(property "Value" "~"
+		(property "Value" ""
 			(at 187.452 42.1132 0)
 			(effects
@@
 			)
 		)
-		(property "Value" "~"
+		(property "Value" ""
 			(at 45.72 110.9472 0)
 			(effects
@@
 			)
 		)
-		(property "Value" "~"
+		(property "Value" ""
 			(at 256.032 141.1732 0)
 			(effects
@@
 			)
 		)
-		(property "Value" "~"
+		(property "Value" ""
 			(at 121.92 65.2272 0)
 			(effects
@@
 			)
 		)
-		(property "Value" "~"
+		(property "Value" ""
 			(at 89.154 156.1592 0)
 			(effects
@@
 			)
 		)
-		(property "Value" "~"
+		(property "Value" ""
 			(at 266.7 88.0872 0)
 			(effects
@@
 			)
 		)
-		(property "Value" "~"
+		(property "Value" ""
 			(at 205.232 151.3332 0)
 			(effects
@@
 			)
 		)
-		(property "Value" "~"
+		(property "Value" ""
 			(at 254 143.9672 0)
 			(effects
@@
 			)
 		)
-		(property "Value" "~"
+		(property "Value" ""
 			(at 38.354 133.2992 0)
 			(effects
@@
 			)
 		)
-		(property "Value" "~"
+		(property "Value" ""
 			(at 48.514 156.1592 0)
 			(effects
@@
 			)
 		)
-		(property "Value" "~"
+		(property "Value" ""
 			(at 261.112 124.6632 0)
 			(effects
@@
 			)
 		)
-		(property "Value" "~"
+		(property "Value" ""
 			(at 139.954 176.4792 0)
 			(effects
@@
 			)
 		)
-		(property "Value" "~"
+		(property "Value" ""
 			(at 205.232 133.5532 0)
 			(effects
@@
 			)
 		)
-		(property "Value" "~"
+		(property "Value" ""
 			(at 249.174 46.9392 0)
 			(effects
@@
 			)
 		)
-		(property "Value" "~"
+		(property "Value" ""
 			(at 271.526 95.4532 0)
 			(effects
@@
 			)
 		)
-		(property "Value" "~"
+		(property "Value" ""
 			(at 172.974 135.8392 0)
 			(effects
@@
 			)
 		)
-		(property "Value" "~"
+		(property "Value" ""
 			(at 231.14 164.2872 0)
 			(effects
@@
 			)
 		)
-		(property "Value" "~"
+		(property "Value" ""
 			(at 165.1 171.9072 0)
 			(effects
@@
 			)
 		)
-		(property "Value" "~"
+		(property "Value" ""
 			(at 28.194 156.1592 0)
 			(effects
@@
 			)
 		)
-		(property "Value" "~"
+		(property "Value" ""
 			(at 35.814 105.3592 0)
 			(effects
@@
 			)
 		)
-		(property "Value" "~"
+		(property "Value" ""
 			(at 78.994 133.2992 0)
 			(effects
@@
 			)
 		)
-		(property "Value" "~"
+		(property "Value" ""
 			(at 38.354 179.0192 0)
 			(effects
@@
 			)
 		)
-		(property "Value" "~"
+		(property "Value" ""
 			(at 187.452 26.8732 0)
 			(effects
@@
 			)
 		)
-		(property "Value" "~"
+		(property "Value" ""
 			(at 68.834 156.1592 0)
 			(effects
@@
 			)
 		)
-		(property "Value" "~"
+		(property "Value" ""
 			(at 233.172 87.8332 0)
 			(effects
@@
 			)
 		)
-		(property "Value" "~"
+		(property "Value" ""
 			(at 48.514 133.2992 0)
 			(effects
@@
 			)
 		)
-		(property "Value" "~"
+		(property "Value" ""
 			(at 25.654 100.2792 0)
 			(effects
@@
 			)
 		)
-		(property "Value" "~"
+		(property "Value" ""
 			(at 256.032 118.3132 0)
 			(effects
@@
 			)
 		)
-		(property "Value" "~"
+		(property "Value" ""
 			(at 210.312 157.6832 0)
 			(effects
@@
 			)
 		)
-		(property "Value" "~"
+		(property "Value" ""
 			(at 198.374 135.8392 0)
 			(effects
@@
 			)
 		)
-		(property "Value" "~"
+		(property "Value" ""
 			(at 58.674 156.1592 0)
 			(effects
@@
 			)
 		)
-		(property "Value" "~"
+		(property "Value" ""
 			(at 149.86 126.1872 0)
 			(effects
@@
 			)
 		)
-		(property "Value" "~"
+		(property "Value" ""
 			(at 236.22 34.7472 0)
 			(effects
@@
 			)
 		)
-		(property "Value" "~"
+		(property "Value" ""
 			(at 183.134 135.8392 0)
 			(effects
@@
 			)
 		)
-		(property "Value" "~"
+		(property "Value" ""
 			(at 258.572 176.9872 0)
 			(effects
@@
 			)
 		)
-		(property "Value" "~"
+		(property "Value" ""
 			(at 205.994 176.4792 0)
 			(effects
@@
 			)
 		)
-		(property "Value" "~"
+		(property "Value" ""
 			(at 89.154 133.2992 0)
 			(effects
@@
 			)
 		)
-		(property "Value" "~"
+		(property "Value" ""
 			(at 261.112 147.5232 0)
 			(effects
