File: STM32_microcontroller_IOs.kicad_sch (KiCad schematic)
At the start: 31 parts

Commit message: kicad xfer
Parts:
- B4, C43, C44, C67, HW20, JP3, LED1, LED2, LED3, R26, R34, R35, R36, SB10, SB11, SB12, SB13, SB14, SB2, SB3, SB31, SB4, SB5, SB6, SB7, SB8, SB9, U11, U6, X2: value ~ -> (none)
Changed lines of the file:
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@@
 			)
 		)
-		(property "Value" "~"
+		(property "Value" ""
 			(at 238.252 58.6232 0)
 			(effects
@@
 			)
 		)
-		(property "Value" "~"
+		(property "Value" ""
 			(at 139.954 157.4292 0)
 			(effects
@@
 			)
 		)
-		(property "Value" "~"
+		(property "Value" ""
 			(at 238.252 53.5432 0)
 			(effects
@@
 			)
 		)
-		(property "Value" "~"
+		(property "Value" ""
 			(at 241.554 55.8292 0)
 			(effects
@@
 			)
 		)
-		(property "Value" "~"
+		(property "Value" ""
 			(at 66.04 192.2272 0)
 			(effects
@@
 			)
 		)
-		(property "Value" "~"
+		(property "Value" ""
 			(at 147.32 113.4872 0)
 			(effects
@@
 			)
 		)
-		(property "Value" "~"
+		(property "Value" ""
 			(at 238.76 174.4472 0)
 			(effects
@@
 			)
 		)
-		(property "Value" "~"
+		(property "Value" ""
 			(at 266.7 164.2872 90)
 			(effects
@@
 			)
 		)
-		(property "Value" "~"
+		(property "Value" ""
 			(at 91.694 45.6692 0)
 			(effects
@@
 			)
 		)
-		(property "Value" "~"
+		(property "Value" ""
 			(at 88.392 43.3832 0)
 			(effects
@@
 			)
 		)
-		(property "Value" "~"
+		(property "Value" ""
 			(at 91.694 50.7492 0)
 			(effects
@@
 			)
 		)
-		(property "Value" "~"
+		(property "Value" ""
 			(at 139.954 159.9692 0)
 			(effects
@@
 			)
 		)
-		(property "Value" "~"
+		(property "Value" ""
 			(at 58.42 171.9072 0)
 			(effects
@@
 			)
 		)
-		(property "Value" "~"
+		(property "Value" ""
 			(at 162.56 159.2072 0)
 			(effects
@@
 			)
 		)
-		(property "Value" "~"
+		(property "Value" ""
 			(at 210.312 143.7132 0)
 			(effects
@@
 			)
 		)
-		(property "Value" "~"
+		(property "Value" ""
 			(at 241.554 60.9092 0)
 			(effects
@@
 			)
 		)
-		(property "Value" "~"
+		(property "Value" ""
 			(at 14.732 123.9012 0)
 			(effects
@@
 			)
 		)
-		(property "Value" "~"
+		(property "Value" ""
 			(at 241.554 48.2092 0)
 			(effects
@@
 			)
 		)
-		(property "Value" "~"
+		(property "Value" ""
 			(at 139.954 144.7292 0)
 			(effects
@@
 			)
 		)
-		(property "Value" "~"
+		(property "Value" ""
 			(at 218.694 166.3192 0)
 			(effects
@@
 			)
 		)
-		(property "Value" "~"
+		(property "Value" ""
 			(at 71.12 187.1472 0)
 			(effects
@@
 			)
 		)
-		(property "Value" "~"
+		(property "Value" ""
 			(at 40.64 143.9672 0)
 			(effects
@@
 			)
 		)
-		(property "Value" "~"
+		(property "Value" ""
 			(at 139.954 147.2692 0)
 			(effects
@@
 			)
 		)
-		(property "Value" "~"
+		(property "Value" ""
 			(at 218.44 141.4272 0)
 			(effects
@@
 			)
 		)
-		(property "Value" "~"
+		(property "Value" ""
 			(at 68.072 169.3672 0)
 			(effects
@@
 			)
 		)
-		(property "Value" "~"
+		(property "Value" ""
 			(at 241.554 50.7492 0)
 			(effects
@@
 			)
 		)
-		(property "Value" "~"
+		(property "Value" ""
 			(at 14.732 151.8412 0)
 			(effects
@@
 			)
 		)
-		(property "Value" "~"
+		(property "Value" ""
 			(at 240.792 143.2052 0)
 			(effects
@@
 			)
 		)
-		(property "Value" "~"
+		(property "Value" ""
 			(at 58.42 182.0672 0)
 			(effects
@@
 			)
 		)
-		(property "Value" "~"
+		(property "Value" ""
 			(at 58.42 192.2272 0)
 			(effects
@@
 			)
 		)
-		(property "Value" "~"
+		(property "Value" ""
 			(at 88.392 48.4632 0)
 			(effects
