File: STM32_microcontroller_RF.kicad_sch (KiCad schematic)
At the start: 83 parts, among them X4 NT2016SF

Commit message: kicad xfer
Parts:
- C13, C14, C16, C19, C2, C20, C21, C24, C25, C30, C35, C37, C38, C5, C6, C71, C72, C73, C74, C76, C77, C78, C79, C8, C80, C82, C85, CN12, CN13, L10, L12, L13, L2, L4, L8, L9, R27, R28, R29, R32, R33, R37, R38, R39, R40, R41, SB18, SB20, SB22, SB23, SC1, SC3, SC4, SC5, SC6, SC7, U1, U3, U4, U6, X3: value ~ -> (none)
Changed lines of the file:
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@@
 			)
 		)
-		(property "Value" "~"
+		(property "Value" ""
 			(at 101.6 266.5222 0)
 			(effects
@@
 			)
 		)
-		(property "Value" "~"
+		(property "Value" ""
 			(at 83.82 266.5222 0)
 			(effects
@@
 			)
 		)
-		(property "Value" "~"
+		(property "Value" ""
 			(at 17.78 251.7902 0)
 			(effects
@@
 			)
 		)
-		(property "Value" "~"
+		(property "Value" ""
 			(at 370.078 136.4742 0)
 			(effects
@@
 			)
 		)
-		(property "Value" "~"
+		(property "Value" ""
 			(at 111.76 70.9422 0)
 			(effects
@@
 			)
 		)
-		(property "Value" "~"
+		(property "Value" ""
 			(at 39.116 83.1342 0)
 			(effects
@@
 			)
 		)
-		(property "Value" "~"
+		(property "Value" ""
 			(at 312.42 136.9822 0)
 			(effects
@@
 			)
 		)
-		(property "Value" "~"
+		(property "Value" ""
 			(at 256.794 182.1942 0)
 			(effects
@@
 			)
 		)
-		(property "Value" "~"
+		(property "Value" ""
 			(at 53.594 70.4342 0)
 			(effects
@@
 			)
 		)
-		(property "Value" "~"
+		(property "Value" ""
 			(at 152.654 45.0342 0)
 			(effects
@@
 			)
 		)
-		(property "Value" "~"
+		(property "Value" ""
 			(at 238.76 177.6222 0)
 			(effects
@@
 			)
 		)
-		(property "Value" "~"
+		(property "Value" ""
 			(at 292.1 263.9822 0)
 			(effects
@@
 			)
 		)
-		(property "Value" "~"
+		(property "Value" ""
 			(at 358.14 136.9822 0)
 			(effects
@@
 			)
 		)
-		(property "Value" "~"
+		(property "Value" ""
 			(at 309.372 157.3022 0)
 			(effects
@@
 			)
 		)
-		(property "Value" "~"
+		(property "Value" ""
 			(at 152.654 227.9142 0)
 			(effects
@@
 			)
 		)
-		(property "Value" "~"
+		(property "Value" ""
 			(at 142.24 203.0222 0)
 			(effects
@@
 			)
 		)
-		(property "Value" "~"
+		(property "Value" ""
 			(at 155.194 172.0342 0)
 			(effects
@@
 			)
 		)
-		(property "Value" "~"
+		(property "Value" ""
 			(at 207.772 165.1762 0)
 			(effects
@@
 			)
 		)
-		(property "Value" "~"
+		(property "Value" ""
 			(at 78.232 108.2802 0)
 			(effects
@@
 			)
 		)
-		(property "Value" "~"
+		(property "Value" ""
 			(at 99.314 139.0142 0)
 			(effects
@@
 			)
 		)
-		(property "Value" "~"
+		(property "Value" ""
 			(at 327.914 266.0142 0)
 			(effects
@@
 			)
 		)
-		(property "Value" "~"
+		(property "Value" ""
 			(at 83.82 253.8222 0)
 			(effects
@@
 			)
 		)
-		(property "Value" "~"
+		(property "Value" ""
 			(at 221.234 182.1942 0)
 			(effects
@@
 			)
 		)
-		(property "Value" "~"
+		(property "Value" ""
 			(at 101.6 253.8222 0)
 			(effects
@@
 			)
 		)
-		(property "Value" "~"
+		(property "Value" ""
 			(at 160.02 164.9222 0)
 			(effects
@@
 			)
 		)
-		(property "Value" "~"
+		(property "Value" ""
 			(at 13.97 131.3942 0)
 			(effects
@@
 			)
 		)
-		(property "Value" "~"
+		(property "Value" ""
 			(at 43.18 124.2822 0)
 			(effects
@@
 			)
 		)
-		(property "Value" "~"
+		(property "Value" ""
 			(at 228.092 175.3362 0)
 			(effects
@@
 			)
 		)
-		(property "Value" "~"
+		(property "Value" ""
 			(at 60.452 225.1202 0)
 			(effects
@@
 			)
 		)
-		(property "Value" "~"
+		(property "Value" ""
 			(at 66.04 266.5222 0)
 			(effects
@@
 			)
 		)
-		(property "Value" "~"
+		(property "Value" ""
 			(at 220.472 258.9022 0)
 			(effects
@@
 			)
 		)
-		(property "Value" "~"
+		(property "Value" ""
 			(at 277.114 266.0142 0)
 			(effects
@@
 			)
 		)
-		(property "Value" "~"
+		(property "Value" ""
 			(at 312.674 141.5542 0)
 			(effects
@@
 			)
 		)
-		(property "Value" "~"
+		(property "Value" ""
 			(at 54.61 52.6542 0)
 			(effects
@@
 			)
 		)
-		(property "Value" "~"
+		(property "Value" ""
 			(at 327.66 111.5822 0)
 			(effects
@@
 			)
 		)
-		(property "Value" "~"
+		(property "Value" ""
 			(at 14.986 228.1682 0)
 			(effects
@@
 			)
 		)
-		(property "Value" "~"
+		(property "Value" ""
 			(at 85.852 52.4002 0)
 			(effects
@@
 			)
 		)
-		(property "Value" "~"
+		(property "Value" ""
 			(at 340.614 111.0742 0)
 			(effects
@@
 			)
 		)
-		(property "Value" "~"
+		(property "Value" ""
 			(at 15.494 50.1142 0)
 			(effects
@@
 			)
 		)
-		(property "Value" "~"
+		(property "Value" ""
 			(at 88.9 236.0422 0)
 			(effects
@@
 			)
 		)
-		(property "Value" "~"
+		(property "Value" ""
 			(at 66.04 253.8222 0)
 			(effects
@@
 			)
 		)
-		(property "Value" "~"
+		(property "Value" ""
 			(at 14.986 263.7282 0)
 			(effects
@@
 			)
 		)
-		(property "Value" "~"
+		(property "Value" ""
 			(at 198.374 182.1942 0)
 			(effects
@@
 			)
 		)
-		(property "Value" "~"
+		(property "Value" ""
 			(at 78.232 103.2002 0)
 			(effects
@@
 			)
 		)
-		(property "Value" "~"
+		(property "Value" ""
 			(at 183.134 45.0342 0)
 			(effects
@@
 			)
 		)
-		(property "Value" "~"
+		(property "Value" ""
 			(at 155.194 141.5542 0)
 			(effects
@@
 			)
 		)
-		(property "Value" "~"
+		(property "Value" ""
 			(at 69.596 83.1342 0)
 			(effects
@@
 			)
 		)
-		(property "Value" "~"
+		(property "Value" ""
 			(at 28.194 50.1142 0)
 			(effects
@@
 			)
 		)
-		(property "Value" "~"
+		(property "Value" ""
 			(at 83.312 35.3822 0)
 			(effects
@@
 			)
 		)
-		(property "Value" "~"
+		(property "Value" ""
 			(at 236.474 45.0342 0)
 			(effects
@@
 			)
 		)
-		(property "Value" "~"
+		(property "Value" ""
 			(at 169.926 218.0082 0)
 			(effects
@@
 			)
 		)
-		(property "Value" "~"
+		(property "Value" ""
 			(at 302.514 45.0342 0)
 			(effects
@@
 			)
 		)
-		(property "Value" "~"
+		(property "Value" ""
 			(at 65.532 37.1602 0)
 			(effects
@@
 			)
 		)
-		(property "Value" "~"
+		(property "Value" ""
 			(at 142.24 195.4022 0)
 			(effects
@@
 			)
 		)
-		(property "Value" "~"
+		(property "Value" ""
 			(at 330.454 45.0342 0)
 			(effects
@@
 			)
 		)
-		(property "Value" "~"
+		(property "Value" ""
 			(at 362.966 268.8082 0)
 			(effects
@@
 			)
 		)
-		(property "Value" "~"
+		(property "Value" ""
 			(at 84.074 139.0142 0)
 			(effects
@@
 			)
 		)
-		(property "Value" "~"
+		(property "Value" ""
 			(at 96.012 93.2942 0)
 			(effects
@@
 			)
 		)
-		(property "Value" "~"
+		(property "Value" ""
 			(at 60.452 222.5802 0)
 			(effects
@@
 			)
 		)
-		(property "Value" "~"
+		(property "Value" ""
 			(at 118.872 157.3022 0)
 			(effects
@@
 			)
 		)
-		(property "Value" "~"
+		(property "Value" ""
 			(at 59.436 207.5942 0)
 			(effects
@@
 			)
 		)
-		(property "Value" "~"
+		(property "Value" ""
 			(at 343.154 141.5542 0)
 			(effects
