File: radioboard_dev/STM32_microcontroller_RF.kicad_sch (KiCad schematic)
At the start: 83 parts, among them X4 NT2016SF

Commit message: added components
Parts:
- removed CN13: (no value), CON_988-JIUBABA_PHFS25-11-02-G0B115-T-1, symbol MB1389-altium-import:U_STM32_microcontroller_RF_0_Header 2x1
- removed HW103: Daughter_Board, SHIELD_RF_ST-CUSTOM_17P2X17P2_H3, symbol MB1389-altium-import:U_STM32_microcontroller_RF_0_Daughter_Board
- removed R32, R33, R37, R38, R39, R40: (no value), R0402, symbol MB1389-altium-import:U_STM32_microcontroller_RF_2_Resistor
- removed SB18: (no value), SOLDER-BRIDGE_R0603-0R, symbol MB1389-altium-import:U_STM32_microcontroller_RF_3_SB_ON
- removed SB20, SB22, SB23: (no value), SOLDER-BRIDGE_R0603-0R, symbol MB1389-altium-import:U_STM32_microcontroller_RF_1_SB_ON
- removed U1: (no value), ICC_TSNP-9-3_1P1X1P1_P040, symbol MB1389-altium-import:U_STM32_microcontroller_RF_0_BGS13S4N9
- added U8: BGS13SN8E6327XTSA1, parts:TSNP-8-1_INF, symbol BGS13SN8E6327XTSA1:BGS13SN8E6327XTSA1
- C11, C12, C15, C17, C22, C27, C31, C7, C92, C93, C97: footprint C0402 -> parts:C0402
- C13, C14, C16, C19, C2, C20, C21, C24, C25, C30, C37, C38, C5, C6, C71, C72, C73, C74, C76, C77, C78, C79, C8, C80, C82: value (none) -> ~; footprint C0402 -> parts:C0402
- C35, C85: value (none) -> ~; footprint C0603 -> parts:C0603
- CN12: value (none) -> ~; footprint CON_SAMTEC_SMA-J-P-X-ST-EM1 -> parts:CON_SAMTEC_SMA-J-P-X-ST-EM1
- L10, L2, L4, L9: value (none) -> ~; footprint IND_0402_MURATA_LQW15AN_H0P5 -> parts:IND_0402_MURATA_LQW15AN_H0P5
- L11, L3, L5, L6, L7: footprint IND_0402_MURATA_LQW15AN_H0P5 -> parts:IND_0402_MURATA_LQW15AN_H0P5
- L12: value (none) -> ~; footprint IND_0402_MURATA_BLM15H_H0P5 -> parts:IND_0402_MURATA_BLM15H_H0P5
- L13: value (none) -> ~; footprint IND_TDK_MLZ2012M150W -> parts:IND_TDK_MLZ2012M150W
- L8: value (none) -> ~; footprint IND_0402_MURATA_LQW15AN2N4C00X -> parts:IND_0402_MURATA_LQW15AN2N4C00X
- R2: footprint R0402 -> parts:R0402
- R27, R28, R29, R41: value (none) -> ~; footprint R0402 -> parts:R0402
- SC1, SC3, SC4, SC5, SC6, SC7: value (none) -> ~
- U3, U4: value (none) -> ~; footprint ICC_SOT886_XSON6 -> parts:ICC_SOT886_XSON6
- U6: value (none) -> ~; footprint ICC_UFBGA73_5X5_P050 -> parts:QFN50P700X700X60-49N
- X3: value (none) -> ~; footprint CRY_NX2016SA_4P -> parts:CRY_NX2016SA_4P
- X4: footprint CRY_NDK_NT2016SB_4P -> parts:CRY_NDK_NT2016SB_4P
Connections:
- net PB0 is gone; now on net PB0_VDD_TCXO: U6.F6 (PB0-VDD_TCXO)
- net VDD_RF is gone; now on net VDDRF: C35.2, C37.1, U6.A2 (VDDSMPS)
- net FE_CTRL3: now also R29.2
- net GND: now also U8.8 (DGND)
- net VDDRF: now also U3.3 (Y0)
- net VDDRF1V55: now also C85.2, L13.1, U3.1 (Y1), U6.B2 (VFBSMPS)
- net XTA: now also C30.2, X3.1
- net at C38.2, X3.3: now also U6.F8 (OSC_OUT)
- net at U6.B1 (VLXSMPS): now also L13.2
- net at C72.2, R27.2: now also U8.3 (V1)
- net at C8.2, L4.2: now also U8.4 (RF3)
- net at C73.2, R29.1: now also U8.1 (VDD)
- net at C17.2, C20.2: now also U8.5 (RF1)
- net at C2.2: now also U8.6 (RFin)
- net at C7.2, L3.2: now also U8.7 (RF2)
- net at C71.2, R28.2: now also U8.2 (V2)
Other:
- note added: "Author: Forrest Milner, Summer 2024"
- note added: "high power"
- note added: "low power"
- note added: "radioboard"
- note removed: "${BOARD_ASSEMBLY_REVISION}"
- note removed: "${BOARD_DOCUMENT_DATE}"
- note removed: "${BOARD_NAME}"
- note removed: "${BOARD_PCB_REVISION}"
- note removed: "${BOARD_REFERENCE}"
- note removed: "${VARIANTNAME}"
- note removed: "Variant:"

Commit message: finish schematic and clear pcb
Parts:
- removed SC1, SC3, SC4, SC5, SC6, SC7: ~, CLIP_HARWIN_S0951-46R, symbol MB1389-altium-import:U_STM32_microcontroller_RF_0_Shield-clip_S0951-46R
- removed SC2: Shield-clip_S0951-46R, symbol MB1389-altium-import:U_STM32_microcontroller_RF_0_Shield-clip_S0951-46R
- removed SC8, SC9: Shield-clip_S0981-46R, symbol MB1389-altium-import:U_STM32_microcontroller_RF_0_Shield-clip_S0951-46R
- removed U6: ~, parts:QFN50P700X700X60-49N, symbol MB1389-altium-import:U_STM32_microcontroller_RF_0_STM32WL5x_BGA73
Connections:
- net OSC_OUT: now reaches C38.2, X3.3
- net VLXSMPS: now reaches L13.2
- net RFO_LP: now reaches L10.1
- net VR_PA: now reaches C74.2, C76.2, C92.2, U4.4 (Z)
- net RFO_HP: now reaches L9.1
- net XTA renamed OSC_IN
Other:
- note removed: "Shield clips for metal RF cavity"

Commit message: footprints
Parts:
- X4: ALTERNATE_MANUFACTURER N/A -> (none); ALTERNATE_MANUFACTURER_PART_NUMBER N/A -> (none); ALTIUM_VALUE 32MHz -> (none); COMPONENTLINK1DESCRIPTION Part_Information -> (none); COMPONENTLINK1URL http://tunmcdsvn.tun.st.com/Component_Datasheet_Library/Tru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 -> (none); MANUFACTURER NDK -> (none); MANUFACTURER_PART_NUMBER NT2016SF-32M-END5875A -> (none); ORDER_CODE_DIGIKEY N/A -> (none); ORDER_CODE_FARNELL N/A -> (none); ORDER_CODE_RS N/A -> (none); PACKAGE 2016 size -> (none); PART_PREFERENCE Recommended -> (none); PART_TYPE Crystal_Osc -> (none); STATUS Checked -> (none)
Changed lines of the file:
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@@
 		)
 		(property "Description" "NT2016SF-32M-END5875A"
-			(at 25.4 152.4 0)
+			(at 33.274 164.592 0)
 			(effects
 				(font
 					(size 1.27 1.27)
 				)
-				(hide yes)
 			)
 		)
@@
 			(effects
 				(font
-					(size 1.27 1.27)
-				)
-				(justify left bottom)
-				(hide yes)
-			)
-		)
-		(property "ALTIUM_VALUE" "32MHz"
-			(at 35.56 152.4 0)
-			(effects
-				(font
-					(size 1.27 1.27)
-				)
-				(justify left bottom)
-			)
-		)
-		(property "STATUS" "Checked"
-			(at 19.812 147.32 0)
-			(effects
-				(font
-					(size 1.27 1.27)
-				)
-				(justify left bottom)
-				(hide yes)
-			)
-		)
-		(property "PART_PREFERENCE" "Recommended"
-			(at 19.812 147.32 0)
-			(effects
-				(font
-					(size 1.27 1.27)
-				)
-				(justify left bottom)
-				(hide yes)
-			)
-		)
-		(property "PART_TYPE" "Crystal_Osc"
-			(at 19.812 147.32 0)
-			(effects
-				(font
-					(size 1.27 1.27)
-				)
-				(justify left bottom)
-				(hide yes)
-			)
-		)
-		(property "MANUFACTURER" "NDK"
-			(at 19.812 147.32 0)
-			(effects
-				(font
-					(size 1.27 1.27)
-				)
-				(justify left bottom)
-				(hide yes)
-			)
-		)
-		(property "MANUFACTURER_PART_NUMBER" "NT2016SF-32M-END5875A"
-			(at 20.32 165.1 0)
-			(effects
-				(font
-					(size 1.27 1.27)
-				)
-				(justify left bottom)
-			)
-		)
-		(property "ALTERNATE_MANUFACTURER" "N/A"
-			(at 19.812 147.32 0)
-			(effects
-				(font
-					(size 1.27 1.27)
-				)
-				(justify left bottom)
-				(hide yes)
-			)
-		)
-		(property "ALTERNATE_MANUFACTURER_PART_NUMBER" "N/A"
-			(at 19.812 147.32 0)
-			(effects
-				(font
-					(size 1.27 1.27)
-				)
-				(justify left bottom)
-				(hide yes)
-			)
-		)
-		(property "PACKAGE" "2016 size"
-			(at 19.812 147.32 0)
-			(effects
-				(font
-					(size 1.27 1.27)
-				)
-				(justify left bottom)
-				(hide yes)
-			)
-		)
-		(property "COMPONENTLINK1DESCRIPTION" "Part_Information"
-			(at 19.812 147.32 0)
-			(effects
-				(font
-					(size 1.27 1.27)
-				)
-				(justify left bottom)
-				(hide yes)
-			)
-		)
-		(property "COMPONENTLINK1URL" "http://tunmcdsvn.tun.st.com/Component_Datasheet_Library/Trunk/Crystal_Osc/NDK_NT2016SF%2032MHz%20END5875A%20(ETS10B-12472)/"
-			(at 19.812 147.32 0)
-			(effects
-				(font
-					(size 1.27 1.27)
-				)
-				(justify left bottom)
-				(hide yes)
-			)
-		)
-		(property "ORDER_CODE_DIGIKEY" "N/A"
-			(at 19.812 147.32 0)
-			(effects
-				(font
-					(size 1.27 1.27)
-				)
-				(justify left bottom)
-				(hide yes)
-			)
-		)
-		(property "ORDER_CODE_FARNELL" "N/A"
-			(at 19.812 147.32 0)
-			(effects
-				(font
-					(size 1.27 1.27)
-				)
-				(justify left bottom)
-				(hide yes)
-			)
-		)
-		(property "ORDER_CODE_RS" "N/A"
-			(at 19.812 147.32 0)
-			(effects
-				(font

Commit message: all footprints done
Parts:
- removed X3: ~, parts:CRY_NX2016SA_4P, symbol MB1389-altium-import:U_STM32_microcontroller_RF_0_XTAL_4_PINS
- removed X4: NT2016SF, parts:CRY_NDK_NT2016SB_4P, symbol MB1389-altium-import:U_STM32_microcontroller_RF_0_NT2016SB
- added XTAL1: NX2016SA-32M-EXS00A-CS06465, parts:NX2016SA_NDK, symbol NX2016SA_NDK:NX2016SA-32M-EXS00A-CS06465
- added Y1: ECS-TXO-25CSMV-320-DY-TR, parts:OSC_ECS-TXO-25CSMV-320-DY-TR, symbol ECS-TXO-25CSMV-320-DY-TR:ECS-TXO-25CSMV-320-DY-TR
- L12: footprint parts:IND_0402_MURATA_BLM15H_H0P5 -> Inductor_SMD:L_0402_1005Metric
- L13: footprint parts:IND_TDK_MLZ2012M150W -> Inductor_SMD:L_0805_2012Metric
Connections:
- net GND: now also XTAL1.2, XTAL1.4, Y1.1 (TRI_STATE), Y1.2 (GND)
- net OSC_IN: now also XTAL1.1
- net OSC_OUT: now also XTAL1.3
- net at R2.1: now also Y1.3 (OUTPUT)
- net at C27.2, L12.1: now also Y1.4 (VDD)
Other:
- note removed: "32 MHz"
- moved on the sheet: C27, C31, L12, R2, R41

Commit message: changed parts to 400MHz version
Parts:
- removed C13, C16: ~, parts:C0402, symbol MB1389-altium-import:U_STM32_microcontroller_RF_2_Capacitor
- removed C17, C22, C93, C97: Capacitor, parts:C0402, symbol MB1389-altium-import:U_STM32_microcontroller_RF_1_Capacitor
- removed C21, C24, C25, C78, C80, C82: ~, parts:C0402, symbol MB1389-altium-import:U_STM32_microcontroller_RF_1_Capacitor
- removed C92: Capacitor, parts:C0402, symbol MB1389-altium-import:U_STM32_microcontroller_RF_2_Capacitor
- removed L5, L6: Inductor, parts:IND_0402_MURATA_LQW15AN_H0P5, symbol MB1389-altium-import:U_STM32_microcontroller_RF_0_Inductor
- removed R41: ~, parts:R0402, symbol MB1389-altium-import:U_STM32_microcontroller_RF_0_Resistor
- added C13: Capacitor, parts:C0402, symbol MB1389-altium-import:U_STM32_microcontroller_RF_0_Capacitor
- added C16: 3.6 pF, Capacitor_SMD:C_0402_1005Metric, symbol MB1389-altium-import:U_STM32_microcontroller_RF_0_Capacitor
- added C24, C25, C78, C80, C82: 68pF, Capacitor_SMD:C_0402_1005Metric, symbol MB1389-altium-import:U_STM32_microcontroller_RF_0_Capacitor
- added L5: 6.8nH, Inductor_SMD:L_0402_1005Metric, symbol MB1389-altium-import:U_STM32_microcontroller_RF_1_Inductor
- added L6: 8.2nH, Inductor_SMD:L_0402_1005Metric, symbol MB1389-altium-import:U_STM32_microcontroller_RF_1_Inductor
- added R5, R6: 0, Resistor_SMD:R_0402_1005Metric, symbol Device:R_US
- C11: value Capacitor -> 15 pF; footprint parts:C0402 -> Capacitor_SMD:C_0402_1005Metric; ALTIUM_VALUE 5.6pF -> (none); COMPONENTLINK1DESCRIPTION Datasheet -> (none); COMPONENTLINK1URL http://tunmcdsvn.tun.st.com/Component_Datasheet_Library/Tru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 -> (none); INTERNAL_PART_NUMBER MCD-01374 -> (none); MANUFACTURER YAGEO -> (none); MANUFACTURER_PART_NUMBER CC0402BRNPO9BN5R6 -> (none); ORDER_CODE_DIGIKEY 311-1625-1-ND -> (none); ORDER_CODE_FARNELL N/A -> (none); ORDER_CODE_RS N/A -> (none); PACKAGE C0402 -> (none); PART_PREFERENCE Recommended -> (none); PART_TYPE Capacitor -> (none); STATUS Released -> (none)
- C14: value ~ -> 15 pF; footprint parts:C0402 -> Capacitor_SMD:C_0402_1005Metric; ALTIUM_VALUE 3.3pF -> (none); COMPONENTLINK1DESCRIPTION Datasheet -> (none); COMPONENTLINK1URL http://tunmcdsvn.tun.st.com/Component_Datasheet_Library/Tru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 -> (none); ECCN_EU n/a -> (none); ECCN_US n/a -> (none); INTERNAL_PART_NUMBER MCD-01775 -> (none); MANUFACTURER YAGEO -> (none); MANUFACTURER_PART_NUMBER CC0402BRNPO9BN3R3 -> (none); PACKAGE C0402 -> (none); PART_TYPE Capacitor -> (none); PROVIDED_BY SUBCO -> (none); STATUS Checked -> (none)
- C15: value Capacitor -> 4.3 pF; footprint parts:C0402 -> Capacitor_SMD:C_0402_1005Metric; ALTIUM_VALUE 2.2pF -> (none); COMPONENTLINK1DESCRIPTION Datasheet -> (none); COMPONENTLINK1URL http://tunmcdsvn.tun.st.com/Component_Datasheet_Library/Tru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 -> (none); INTERNAL_PART_NUMBER MCD-01773 -> (none); MANUFACTURER YAGEO -> (none); MANUFACTURER_PART_NUMBER CC0402BRNPO9BN2R2 -> (none); ORDER_CODE_DIGIKEY 311-1618-1-ND -> (none); ORDER_CODE_FARNELL N/A -> (none); ORDER_CODE_RS N/A -> (none); PACKAGE C0402 -> (none); PART_PREFERENCE Recommended -> (none); PART_TYPE Capacitor -> (none); STATUS Released -> (none)
- C19: value ~ -> 4.7pF; ALTIUM_VALUE 2.7pF -> (none); COMPONENTLINK1DESCRIPTION Datasheet -> (none); COMPONENTLINK1URL http://tunmcdsvn.tun.st.com/Component_Datasheet_Library/Tru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 -> (none); ECCN_EU n/a -> (none); ECCN_US n/a -> (none); INTERNAL_PART_NUMBER MCD-01774 -> (none); MANUFACTURER YAGEO -> (none); MANUFACTURER_PART_NUMBER CC0402BRNPO9BN2R7 -> (none); PACKAGE C0402 -> (none); PART_TYPE Capacitor -> (none); PROVIDED_BY SUBCO -> (none); STATUS Checked -> (none)
- C2: value ~ -> 68pF; footprint parts:C0402 -> Capacitor_SMD:C_0402_1005Metric; ALTIUM_VALUE 33pF -> (none); COMPONENTLINK1DESCRIPTION Datasheet -> (none); COMPONENTLINK1URL http://tunmcdsvn.tun.st.com/Component_Datasheet_Library/Tru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 -> (none); ECCN_EU n/a -> (none); ECCN_US n/a -> (none); INTERNAL_PART_NUMBER MCD-01784 -> (none); MANUFACTURER YAGEO -> (none); MANUFACTURER_PART_NUMBER CC0402GRNPO9BN330 -> (none); PACKAGE C0402 -> (none); PART_TYPE Capacitor -> (none); PROVIDED_BY SUBCO -> (none); STATUS Checked -> (none)
- C30, C38, XTAL1: now not fitted; now left out of the parts list
- C5, C6: value ~ -> 6.8pF; ALTIUM_VALUE 3.3pF -> (none); COMPONENTLINK1DESCRIPTION Datasheet -> (none); COMPONENTLINK1URL http://tunmcdsvn.tun.st.com/Component_Datasheet_Library/Tru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 -> (none); ECCN_EU n/a -> (none); ECCN_US n/a -> (none); INTERNAL_PART_NUMBER MCD-01775 -> (none); MANUFACTURER YAGEO -> (none); MANUFACTURER_PART_NUMBER CC0402BRNPO9BN3R3 -> (none); PACKAGE C0402 -> (none); PART_TYPE Capacitor -> (none); PROVIDED_BY SUBCO -> (none); STATUS Checked -> (none)
- C7: ALTERNATE_MANUFACTURER N/A -> (none); ALTERNATE_MANUFACTURER_PART_NUMBER N/A -> (none); ALTIUM_VALUE 1.2pF -> 5.6pF; BMS_PART_NUMBER N/A -> (none); COMPONENTLINK1URL http://tunmcdsvn.tun.st.com/Component_Datasheet_Library/Trunk/Capacitors/MURATA_Chip_Monolithic_Ceramic_Capacitors -> http://tunmcdsvn.tun.st.com/Component_Datasheet_Library/Trunk/Capacitors/Yageo_Capacitor_NP0_16V-to-50V; INTERNAL_PART_NUMBER MCD-02065 -> MCD-01374; MANUFACTURER MURATA -> YAGEO; MANUFACTURER_PART_NUMBER GJM1555C1H1R2WB01D -> CC0402BRNPO9BN5R6; ORDER_CODE_DIGIKEY 490-11195-2-ND -> 311-1625-1-ND; ORDER_CODE_FARNELL 2781428 -> N/A; ORDER_CODE_RS 846-7246 -> N/A; STATUS Checked -> Released
- C8: value ~ -> Capacitor; ALTIUM_VALUE 1.3pF -> 5.6pF; ECCN_EU n/a -> (none); ECCN_US n/a -> (none); INTERNAL_PART_NUMBER MCD-01772 -> MCD-01374; MANUFACTURER_PART_NUMBER CC0402BRNPO9BN1R3 -> CC0402BRNPO9BN5R6; ORDER_CODE_DIGIKEY (none) -> 311-1625-1-ND; ORDER_CODE_FARNELL (none) -> N/A; ORDER_CODE_RS (none) -> N/A; PART_PREFERENCE (none) -> Recommended; PROVIDED_BY SUBCO -> (none); STATUS Checked -> Released
- L10: value ~ -> 0R; footprint parts:IND_0402_MURATA_LQW15AN_H0P5 -> Inductor_SMD:L_0402_1005Metric; ALTIUM_VALUE 3.3nH -> (none); COMPONENTLINK1DESCRIPTION Datasheet -> (none); COMPONENTLINK1URL http://tunmcdsvn.tun.st.com/Component_Datasheet_Library/Tru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 -> (none); ECCN_EU n/a -> (none); ECCN_US n/a -> (none); INTERNAL_PART_NUMBER MCD-01761 -> (none); MANUFACTURER MURATA -> (none); MANUFACTURER_PART_NUMBER LQW15AN3N3D10 -> (none); PACKAGE L0402 -> (none); PART_TYPE Inductor -> (none); PROVIDED_BY SUBCO -> (none); STATUS Checked -> (none)
- L11: value Inductor -> 33nH; ALTIUM_VALUE 11nH -> (none); COMPONENTLINK1DESCRIPTION Datasheet -> (none); COMPONENTLINK1URL http://tunmcdsvn.tun.st.com/Component_Datasheet_Library/Tru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 -> (none); ECCN_EU n/a -> (none); ECCN_US n/a -> (none); INTERNAL_PART_NUMBER MCD-01921 -> (none); MANUFACTURER MURATA -> (none); MANUFACTURER_PART_NUMBER LQW15AN11NG00 -> (none); PACKAGE L0402 -> (none); PART_TYPE Inductor -> (none); PROVIDED_BY SUBCO -> (none); STATUS Footprint available -> (none)
- L2: value ~ -> 16nH; footprint parts:IND_0402_MURATA_LQW15AN_H0P5 -> Inductor_SMD:L_0402_1005Metric; ALTIUM_VALUE 8.7nH -> (none); COMPONENTLINK1DESCRIPTION Datasheet -> (none); COMPONENTLINK1URL http://tunmcdsvn.tun.st.com/Component_Datasheet_Library/Tru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 -> (none); ECCN_EU n/a -> (none); ECCN_US n/a -> (none); INTERNAL_PART_NUMBER MCD-01768 -> (none); MANUFACTURER MURATA -> (none); MANUFACTURER_PART_NUMBER LQW15AN8N7H00 -> (none); PACKAGE L0402 -> (none); PART_TYPE Inductor -> (none); PROVIDED_BY SUBCO -> (none); STATUS Checked -> (none)
- L3: value Inductor -> 16nH; footprint parts:IND_0402_MURATA_LQW15AN_H0P5 -> Inductor_SMD:L_0402_1005Metric; ALTIUM_VALUE 8.7nH -> (none); COMPONENTLINK1DESCRIPTION Datasheet -> (none); COMPONENTLINK1URL http://tunmcdsvn.tun.st.com/Component_Datasheet_Library/Tru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 -> (none); INTERNAL_PART_NUMBER MCD-01768 -> (none); MANUFACTURER MURATA -> (none); MANUFACTURER_PART_NUMBER LQW15AN8N7H00 -> (none); PACKAGE L0402 -> (none); PART_PREFERENCE Recommended -> (none); PART_TYPE Inductor -> (none); STATUS Released -> (none)
- L4: value ~ -> 18nH; footprint parts:IND_0402_MURATA_LQW15AN_H0P5 -> Inductor_SMD:L_0402_1005Metric; ALTIUM_VALUE 8.7nH -> (none); COMPONENTLINK1DESCRIPTION Datasheet -> (none); COMPONENTLINK1URL http://tunmcdsvn.tun.st.com/Component_Datasheet_Library/Tru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 -> (none); ECCN_EU n/a -> (none); ECCN_US n/a -> (none); INTERNAL_PART_NUMBER MCD-01768 -> (none); MANUFACTURER MURATA -> (none); MANUFACTURER_PART_NUMBER LQW15AN8N7H00 -> (none); PACKAGE L0402 -> (none); PART_TYPE Inductor -> (none); PROVIDED_BY SUBCO -> (none); STATUS Checked -> (none)
- L7: value Inductor -> 56nH; footprint parts:IND_0402_MURATA_LQW15AN_H0P5 -> Inductor_SMD:L_0402_1005Metric; ALTERNATE_MANUFACTURER N/A -> (none); ALTERNATE_MANUFACTURER_PART_NUMBER N/A -> (none); ALTIUM_VALUE 33nH -> (none); BMS_PART_NUMBER N/A -> (none); COMPONENTLINK1DESCRIPTION Datasheet -> (none); COMPONENTLINK1URL http://tunmcdsvn.tun.st.com/Component_Datasheet_Library/Tru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 -> (none); INTERNAL_PART_NUMBER MCD-02069 -> (none); MANUFACTURER MURATA -> (none); MANUFACTURER_PART_NUMBER LQW15AN33NG00 -> (none); ORDER_CODE_DIGIKEY 490-6804-1-ND -> (none); ORDER_CODE_FARNELL 1762626 -> (none); ORDER_CODE_RS 169-2777 -> (none); PACKAGE L0402 -> (none); PART_PREFERENCE Recommended -> (none); PART_TYPE Inductor -> (none); STATUS Released -> (none)
- L8: value ~ -> 68nH; footprint parts:IND_0402_MURATA_LQW15AN2N4C00X -> Inductor_SMD:L_0402_1005Metric; ALTIUM_VALUE 47nH -> (none); COMPONENTLINK1DESCRIPTION Datasheet -> (none); COMPONENTLINK1URL http://tunmcdsvn.tun.st.com/Component_Datasheet_Library/Tru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 -> (none); ECCN_EU n/a -> (none); ECCN_US n/a -> (none); INTERNAL_PART_NUMBER MCD-01609 -> (none); MANUFACTURER MURATA -> (none); MANUFACTURER_PART_NUMBER LQW15AN47NJ00# -> (none); PACKAGE L0402 -> (none); PART_TYPE Inductor -> (none); PROVIDED_BY SUBCO -> (none); STATUS Footprint available -> (none)
- L9: value ~ -> 0R; footprint parts:IND_0402_MURATA_LQW15AN_H0P5 -> Inductor_SMD:L_0402_1005Metric; ALTIUM_VALUE 3.6nH -> (none); COMPONENTLINK1DESCRIPTION Datasheet -> (none); COMPONENTLINK1URL http://tunmcdsvn.tun.st.com/Component_Datasheet_Library/Tru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 -> (none); ECCN_EU n/a -> (none); ECCN_US n/a -> (none); INTERNAL_PART_NUMBER MCD-01762 -> (none); MANUFACTURER MURATA -> (none); MANUFACTURER_PART_NUMBER LQW15AN3N6C10 -> (none); PACKAGE L0402 -> (none); PART_TYPE Inductor -> (none); PROVIDED_BY SUBCO -> (none); STATUS Checked -> (none)
Connections:
- net GND: now also C24.2, C25.2, C78.1, C80.2, C82.1
- net OSC_IN: now also R5.2; no longer C30.2, XTAL1.1
- net OSC_OUT: now also R6.1; no longer C38.2, XTAL1.3
- net VDDPA: now also C78.2
- net VDDRF: now also C82.2
- net VDDRF1V55: now also C80.1
- net at C15.1, L7.2, L9.2: now also L5.1
- net at C11.2, C12.1, C15.2: now also L5.2
- net at L4.1: now also C13.2
- net at L10.2, L8.2: now also C16.1, L6.1
- net at L8.1, U4.1 (Y1): now also C25.1
- net at C14.2: now also C13.1, C16.2, L6.2
- net at L7.1, U4.3 (Y0): now also C24.1
- new net: C38.2, R6.2, XTAL1.3
- new net: C30.2, R5.1, XTAL1.1

Commit message: done for day
Parts:
- C37: footprint parts:C0402 -> Capacitor_SMD:C_0402_1005Metric
Changed lines of the file:
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@@
 			)
 		)
-		(property "Footprint" "parts:C0402"
+		(property "Footprint" "Capacitor_SMD:C_0402_1005Metric"
 			(at 33.02 53.34 0)
 			(effects

Commit message: pre mass edit of footprints
Parts:
- C8: footprint parts:C0402 -> Capacitor_SMD:C_0402_1005Metric
Changed lines of the file:
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@@
 			)
 		)
-		(property "Footprint" "parts:C0402"
+		(property "Footprint" "Capacitor_SMD:C_0402_1005Metric"
 			(at 256.54 187.96 0)
 			(effects

Commit message: bom changes
Parts:
- C37: value ~ -> 100nF; ALTERNATE_MANUFACTURER MURATA -> (none); ALTERNATE_MANUFACTURER_PART_NUMBER GCM155R71C104KA55D -> (none); ALTIUM_VALUE 100nF -> (none); COMPONENTLINK1DESCRIPTION Datasheet -> (none); COMPONENTLINK1URL http://tunmcdsvn.tun.st.com/Component_Datasheet_Library/Tru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 -> (none); ECCN_EU NEC -> (none); ECCN_US EAR99 -> (none); INTERNAL_PART_NUMBER MCD-00102 -> (none); MANUFACTURER YAGEO -> (none); MANUFACTURER_PART_NUMBER CC0402KRX7R7BB104 -> (none); PACKAGE C0402 -> (none); PART_TYPE Capacitor -> (none); PROVIDED_BY SUBCO -> (none); STATUS Released -> (none)
- CN12: ALTIUM_VALUE SMA-J-P-H-ST-EM1 -> (none); COMPONENTLINK1DESCRIPTION Datasheet -> (none); COMPONENTLINK1URL http://tunmcdsvn.tun.st.com/Component_Datasheet_Library/Tru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 -> (none); ECCN_EU NEC -> (none); ECCN_US EAR99 -> (none); INTERNAL_PART_NUMBER MCD-00279 -> (none); MANUFACTURER SAMTEC -> (none); MANUFACTURER_PART_NUMBER SMA-J-P-H-ST-EM1 -> (none); PART_TYPE Connector -> (none); PROVIDED_BY SUBCO -> (none); STATUS Released -> (none)
- L12: ALTIUM_VALUE 1400R@1GHz -> (none); COMPONENTLINK1DESCRIPTION Datasheet -> (none); COMPONENTLINK1URL http://tunmcdsvn.tun.st.com/Component_Datasheet_Library/Tru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 -> (none); ECCN_EU n/a -> (none); ECCN_US n/a -> (none); INTERNAL_PART_NUMBER MCD-01610 -> (none); MANUFACTURER MURATA -> (none); MANUFACTURER_PART_NUMBER BLM15HG102SN1# -> (none); PACKAGE L0402 -> (none); PART_TYPE Inductor -> (none); PROVIDED_BY SUBCO -> (none); STATUS Footprint available -> (none)
- L13: value ~ -> 15 µH; ALTIUM_VALUE 15uH -> (none); COMPONENTLINK1DESCRIPTION Datasheet -> (none); COMPONENTLINK1URL http://tunmcdsvn.tun.st.com/Component_Datasheet_Library/Tru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 -> (none); ECCN_EU n/a -> (none); ECCN_US n/a -> (none); INTERNAL_PART_NUMBER MCD-01433 -> (none); MANUFACTURER TDK -> (none); MANUFACTURER_PART_NUMBER MLZ2012M150W -> (none); PACKAGE L0805 -> (none); PART_TYPE Inductor -> (none); PROVIDED_BY SUBCO -> (none); STATUS Checked -> (none)
- U3, U4: ALTIUM_VALUE NX3L1T3157GM -> (none); COMPONENTLINK1DESCRIPTION Datasheet -> (none); COMPONENTLINK1URL http://tunmcdsvn.tun.st.com/Component_Datasheet_Library/Tru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 -> (none); ECCN_EU NEC -> (none); ECCN_US EAR99 -> (none); INTERNAL_PART_NUMBER MCD-01514 -> (none); MANUFACTURER NXP -> (none); MANUFACTURER_PART_NUMBER NX3L1T3157GM -> (none); PACKAGE SOT886 -> (none); PART_TYPE IC -> (none); PROVIDED_BY SUBCO -> (none); STATUS Footprint available -> (none)
