File: radioboard_dev/STM32_microcontroller_RF.kicad_sch (KiCad schematic)
At the start: 56 parts, among them U8 BGS13SN8E6327XTSA1, Y1 ECS-TXO-25CSMV-320-DY-TR

Commit message: datasgeers added...
Parts:
- C20: value ~ -> 3.6pF; ALTIUM_VALUE 3.6pF -> (none); COMPONENTLINK1DESCRIPTION Datasheet -> (none); COMPONENTLINK1URL http://tunmcdsvn.tun.st.com/Component_Datasheet_Library/Tru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 -> (none); ECCN_EU n/a -> (none); ECCN_US n/a -> (none); INTERNAL_PART_NUMBER MCD-01776 -> (none); MANUFACTURER YAGEO -> (none); MANUFACTURER_PART_NUMBER CC0402BRNPO9BN3R6 -> (none); PACKAGE C0402 -> (none); PART_TYPE Capacitor -> (none); PROVIDED_BY SUBCO -> (none); STATUS Checked -> (none)
- C27: value Capacitor -> 220nF; ALTIUM_VALUE 220nF -> (none); COMPONENTLINK1URL http://tunmcdsvn.tun.st.com/Component_Datasheet_Library/Tru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 -> (none); INTERNAL_PART_NUMBER MCD-00602 -> (none); MANUFACTURER TDK -> (none); MANUFACTURER_PART_NUMBER C1005X7R1C224K050BE -> (none); ORDER_CODE_DIGIKEY 445-173638-1-ND -> (none); ORDER_CODE_FARNELL N/A -> (none); ORDER_CODE_RS N/A -> (none); PACKAGE C0402 -> (none); PART_PREFERENCE Recommended -> (none); PART_TYPE Capacitor -> (none); STATUS Released -> (none)
- C31: value Capacitor -> 10pF; ALTIUM_VALUE 10pF -> (none); COMPONENTLINK1DESCRIPTION Datasheet -> (none); COMPONENTLINK1URL http://tunmcdsvn.tun.st.com/Component_Datasheet_Library/Tru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 -> (none); INTERNAL_PART_NUMBER MCD-00015 -> (none); MANUFACTURER YAGEO -> (none); MANUFACTURER_PART_NUMBER CC0402JRNPO9BN100 -> (none); PACKAGE C0402 -> (none); PART_PREFERENCE Recommended -> (none); PART_TYPE Capacitor -> (none); STATUS Released -> (none)
- C74: value ~ -> 47nF; ALTIUM_VALUE 47nF -> (none); COMPONENTLINK1DESCRIPTION Datasheet -> (none); COMPONENTLINK1URL http://tunmcdsvn.tun.st.com/Component_Datasheet_Library/Tru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 -> (none); ECCN_EU N/A -> (none); ECCN_US N/A -> (none); INTERNAL_PART_NUMBER MCD-01605 -> (none); MANUFACTURER YAGEO -> (none); MANUFACTURER_PART_NUMBER CC0402KRX7R8BB473 -> (none); PACKAGE C0402 -> (none); PART_TYPE Capacitor -> (none); PROVIDED_BY SUBCO -> (none); STATUS Footprint available -> (none)
- C76: value ~ -> 68pF; ALTIUM_VALUE 68pF -> (none); COMPONENTLINK1DESCRIPTION Datasheet -> (none); COMPONENTLINK1URL http://tunmcdsvn.tun.st.com/Component_Datasheet_Library/Tru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 -> (none); ECCN_EU N/A -> (none); ECCN_US N/A -> (none); INTERNAL_PART_NUMBER MCD-01604 -> (none); MANUFACTURER YAGEO -> (none); MANUFACTURER_PART_NUMBER CC0402JRNPO9BN680 -> (none); PACKAGE C0402 -> (none); PART_TYPE Capacitor -> (none); PROVIDED_BY SUBCO -> (none); STATUS Released -> (none)
- C77: value ~ -> 100nF; ALTERNATE_MANUFACTURER MURATA -> (none); ALTERNATE_MANUFACTURER_PART_NUMBER GCM155R71C104KA55D -> (none); ALTIUM_VALUE 100nF -> (none); COMPONENTLINK1DESCRIPTION Datasheet -> (none); COMPONENTLINK1URL http://tunmcdsvn.tun.st.com/Component_Datasheet_Library/Tru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 -> (none); ECCN_EU NEC -> (none); ECCN_US EAR99 -> (none); INTERNAL_PART_NUMBER MCD-00102 -> (none); MANUFACTURER YAGEO -> (none); MANUFACTURER_PART_NUMBER CC0402KRX7R7BB104 -> (none); PACKAGE C0402 -> (none); PART_TYPE Capacitor -> (none); PROVIDED_BY SUBCO -> (none); STATUS Released -> (none)
- C79: value ~ -> 47pF; ALTIUM_VALUE 47pF -> (none); COMPONENTLINK1DESCRIPTION Datasheet -> (none); COMPONENTLINK1URL http://tunmcdsvn.tun.st.com/Component_Datasheet_Library/Tru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 -> (none); ECCN_EU N/A -> (none); ECCN_US N/A -> (none); INTERNAL_PART_NUMBER MCD-01603 -> (none); MANUFACTURER YAGEO -> (none); MANUFACTURER_PART_NUMBER CC0402JRNPO9BN470 -> (none); PACKAGE C0402 -> (none); PART_TYPE Capacitor -> (none); PROVIDED_BY SUBCO -> (none); STATUS Released -> (none)
- C8: value Capacitor -> 5.6pF; ALTIUM_VALUE 5.6pF -> (none); COMPONENTLINK1DESCRIPTION Datasheet -> (none); COMPONENTLINK1URL http://tunmcdsvn.tun.st.com/Component_Datasheet_Library/Tru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 -> (none); INTERNAL_PART_NUMBER MCD-01374 -> (none); MANUFACTURER YAGEO -> (none); MANUFACTURER_PART_NUMBER CC0402BRNPO9BN5R6 -> (none); ORDER_CODE_DIGIKEY 311-1625-1-ND -> (none); ORDER_CODE_FARNELL N/A -> (none); ORDER_CODE_RS N/A -> (none); PACKAGE C0402 -> (none); PART_PREFERENCE Recommended -> (none); PART_TYPE Capacitor -> (none); STATUS Released -> (none)

Commit message: finished bom
Parts:
- removed R27, R28, R29: ~, parts:R0402, symbol MB1389-altium-import:U_STM32_microcontroller_RF_0_Resistor
- added R27, R28, R29: 220R, parts:R0402, symbol MB1389-altium-import:U_STM32_microcontroller_RF_1_Resistor
- C11, C14: value 15 pF -> 15pF
- C12, C13: value Capacitor -> 68pF; footprint parts:C0402 -> Capacitor_SMD:C_0402_1005Metric; ALTIUM_VALUE 68pF -> (none); MANUFACTURER_PART_NUMBER CC0402JRNPO9BN680 -> (none)
- C15: value 4.3 pF -> 4.3pF
- C16: value 3.6 pF -> 3.6pF
- C20, C76: footprint parts:C0402 -> Capacitor_SMD:C_0402_1005Metric
- C30, C38: value ~ -> 6.8pF; ALTIUM_VALUE 6.8pF -> (none); MANUFACTURER_PART_NUMBER CC0402CRNPO9BN6R8 -> (none)
- C35: value ~ -> 4.7uF; ALTIUM_VALUE 4.7uF -> (none); MANUFACTURER_PART_NUMBER CC0603KRX5R7BB475 -> (none)
- C7: value Capacitor -> 5.6pF; footprint parts:C0402 -> Capacitor_SMD:C_0402_1005Metric; ALTIUM_VALUE 5.6pF -> (none); COMPONENTLINK1DESCRIPTION Datasheet -> (none); COMPONENTLINK1URL http://tunmcdsvn.tun.st.com/Component_Datasheet_Library/Tru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 -> (none); INTERNAL_PART_NUMBER MCD-01374 -> (none); MANUFACTURER YAGEO -> (none); MANUFACTURER_PART_NUMBER CC0402BRNPO9BN5R6 -> (none); ORDER_CODE_DIGIKEY 311-1625-1-ND -> (none); ORDER_CODE_FARNELL N/A -> (none); ORDER_CODE_RS N/A -> (none); PACKAGE C0402 -> (none); PART_PREFERENCE Recommended -> (none); PART_TYPE Capacitor -> (none); STATUS Released -> (none)
- C71, C72, C73: value ~ -> 1nF; ALTIUM_VALUE 1nF -> (none); COMPONENTLINK1DESCRIPTION Datasheet -> (none); COMPONENTLINK1URL http://tunmcdsvn.tun.st.com/Component_Datasheet_Library/Tru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 -> (none); ECCN_EU NEC -> (none); ECCN_US EAR99 -> (none); INTERNAL_PART_NUMBER MCD-00198 -> (none); MANUFACTURER YAGEO -> (none); MANUFACTURER_PART_NUMBER CC0402KRX7R7BB102 -> (none); PACKAGE C0402 -> (none); PART_TYPE Capacitor -> (none); PROVIDED_BY SUBCO -> (none); STATUS Released -> (none)
- C85: value ~ -> 470nF; ALTIUM_VALUE 470nF -> (none); COMPONENTLINK1DESCRIPTION Datasheet -> (none); COMPONENTLINK1URL http://tunmcdsvn.tun.st.com/Component_Datasheet_Library/Tru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 -> (none); ECCN_EU N/A -> (none); ECCN_US N/A -> (none); INTERNAL_PART_NUMBER MCD-01006 -> (none); MANUFACTURER YAGEO -> (none); MANUFACTURER_PART_NUMBER CC0603KRX7R7BB474 -> (none); PACKAGE C0603 -> (none); PART_TYPE Capacitor -> (none); PROVIDED_BY SUBCO -> (none); STATUS Released -> (none)
- L13: value 15 µH -> 15µH
- R2: value Resistor -> 220R; ALTIUM_VALUE 220R -> (none); COMPONENTLINK1DESCRIPTION Datasheet -> (none); COMPONENTLINK1URL http://tunmcdsvn.tun.st.com/Component_Datasheet_Library/Tru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 -> (none); ECCN_EU NEC -> (none); ECCN_US EAR99 -> (none); INTERNAL_PART_NUMBER MCD-00427 -> (none); MANUFACTURER YAGEO -> (none); MANUFACTURER_PART_NUMBER RC0402FR-07220RL -> (none); PACKAGE R0402 -> (none); PART_TYPE Resistor -> (none); PROVIDED_BY SUBCO -> (none); STATUS Released -> (none)
Connections:
- net FE_CTRL1: now also R27.2
- net FE_CTRL2: now also R28.2
- net FE_CTRL3: now also R29.1
- net at C72.2, U8.3 (V1): now also R27.1
- net at C73.2, U8.1 (VDD): now also R29.2
- net at C71.2, U8.2 (V2): now also R28.1
