File: radioboard_dev/STM32_microcontroller_power.kicad_sch (KiCad schematic)
At the start: 18 parts, among them J1 Conn_01x02, J2 Conn_01x02, J4 Conn_01x04, J5 Conn_01x04, J6 Conn_01x04, J9 Conn_01x04, U11 MAX17048G_T10, U12 TPS73733QDRBRQ1, U13 ACS722LLCTR-05AB-T, U5 MCP73831T-2ACI_OT

Commit message: finished bom
Parts:
- C1, C3, C4: value ~ -> 4.7uF; ALTIUM_VALUE 4.7uF -> (none); MANUFACTURER_PART_NUMBER CC0603KRX5R7BB475 -> (none)
- C9: value ~ -> 100nF; ALTIUM_VALUE 100nF -> (none); MANUFACTURER_PART_NUMBER CC0402KRX7R7BB104 -> (none)
- R1: ALTIUM_VALUE 2k -> (none); COMPONENTLINK1DESCRIPTION Datasheet -> (none); COMPONENTLINK1URL http://tunmcdsvn.tun.st.com/Component_Datasheet_Library/Tru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 -> (none); ECCN_EU NEC -> (none); ECCN_US EAR99 -> (none); INTERNAL_PART_NUMBER MCD-00119 -> (none); MANUFACTURER YAGEO -> (none); MANUFACTURER_PART_NUMBER RC0402FR-07100RL -> (none); PACKAGE R0402 -> (none); PART_TYPE Resistor -> (none); PROVIDED_BY SUBCO -> (none); STATUS Released -> (none)
- R3: value ~ -> 270R; ALTIUM_VALUE 270R -> (none); COMPONENTLINK1DESCRIPTION Datasheet -> (none); COMPONENTLINK1URL http://tunmcdsvn.tun.st.com/Component_Datasheet_Library/Tru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 -> (none); ECCN_EU NEC -> (none); ECCN_US EAR99 -> (none); INTERNAL_PART_NUMBER MCD-00441 -> (none); MANUFACTURER YAGEO -> (none); MANUFACTURER_PART_NUMBER RC0402FR-07270RL -> (none); PACKAGE R0402 -> (none); PART_TYPE Resistor -> (none); PROVIDED_BY SUBCO -> (none); STATUS Released -> (none)
