File: radioboard_dev/radioboard_GPS.kicad_sch (KiCad schematic)
At the start: 3 parts, among them J3 Conn_01x04, U1 TPS22917DBVR, U2 SAM-M10Q-00B

Commit message: all footprints done
Other:
- note added: "GPS Module"
- note added: "GPS Switch"
- moved on the sheet: U1
Changed lines of the file:
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@@
 	)
 	(no_connect
-		(at 54.61 38.1)
+		(at 58.42 114.3)
 	)
 	(no_connect
-		(at 54.61 33.02)
+		(at 58.42 109.22)
 	)
 	(wire
@@
 	)
 	(rectangle
-		(start 8.89 12.065)
-		(end 68.58 53.975)
+		(start 14.605 66.04)
+		(end 70.485 132.08)
 		(stroke
 			(width 0)
@@
 		)
 	)
+	(text "GPS Module"
+		(exclude_from_sim no)
+		(at 150.876 55.88 0)
+		(effects
+			(font
+				(size 5.08 5.08)
+			)
+		)
+	)
+	(text "GPS Switch\n"
+		(exclude_from_sim no)
+		(at 39.878 82.296 0)
+		(effects
+			(font
+				(size 5.08 5.08)
+			)
+		)
+	)
 	(global_label "GPSTXD"
 		(shape input)
@@
 	(global_label "VGPS"
 		(shape input)
-		(at 54.61 27.94 0)
+		(at 58.42 104.14 0)
 		(fields_autoplaced yes)
 		(effects
@@
 		)
 		(property "Intersheetrefs" "${INTERSHEET_REFS}"
-			(at 62.4333 27.94 0)
+			(at 66.2433 104.14 0)
 			(effects
 				(font
@@
 	(global_label "GPSPOW"
 		(shape input)
-		(at 24.13 33.02 180)
+		(at 27.94 109.22 180)
 		(fields_autoplaced yes)
 		(effects
@@
 		)
 		(property "Intersheetrefs" "${INTERSHEET_REFS}"
-			(at 13.3434 33.02 0)
+			(at 17.1534 109.22 0)
 			(effects
 				(font
@@
 	(symbol
 		(lib_id "power:+3.3V")
-		(at 24.13 27.94 0)
+		(at 27.94 104.14 0)
 		(unit 1)
 		(exclude_from_sim no)
@@
 		(fields_autoplaced yes)
 		(property "Reference" "#PWR04"
-			(at 24.13 31.75 0)
+			(at 27.94 107.95 0)
 			(effects
 				(font
@@
 		)
 		(property "Value" "+3.3V"
-			(at 24.13 22.86 0)
+			(at 27.94 99.06 0)
 			(effects
 				(font
@@
 		)
 		(property "Footprint" ""
-			(at 24.13 27.94 0)
+			(at 27.94 104.14 0)
 			(effects
 				(font
@@
 		)
 		(property "Datasheet" ""
-			(at 24.13 27.94 0)
+			(at 27.94 104.14 0)
 			(effects
 				(font
@@
 		)
 		(property "Description" "Power symbol creates a global label with name \"+3.3V\""
-			(at 24.13 27.94 0)
+			(at 27.94 104.14 0)
 			(effects
 				(font
@@
 	(symbol
 		(lib_id "MB1389-altium-import:GND_POWER_GROUND")
-		(at 54.61 43.18 0)
+		(at 58.42 119.38 0)
 		(unit 1)
 		(exclude_from_sim no)
@@
 		(dnp no)
 		(property "Reference" "#PWR028"
-			(at 54.61 43.18 0)
+			(at 58.42 119.38 0)
 			(effects
 				(font
@@
 		)
 		(property "Value" "GND"
-			(at 54.61 49.53 0)
+			(at 58.42 125.73 0)
 			(effects
 				(font
@@
 		)
 		(property "Footprint" ""
-			(at 54.61 43.18 0)
+			(at 58.42 119.38 0)
 			(effects
 				(font
@@
 		)
 		(property "Datasheet" ""
-			(at 54.61 43.18 0)
+			(at 58.42 119.38 0)
 			(effects
 				(font
@@
 		)
 		(property "Description" ""
-			(at 54.61 43.18 0)
+			(at 58.42 119.38 0)
 			(effects
 				(font
@@
 	(symbol
 		(lib_id "TPS22917DBVR:TPS22917DBVR")
-		(at 39.37 35.56 0)
+		(at 43.18 111.76 0)
 		(unit 1)
 		(exclude_from_sim no)
@@
 		(fields_autoplaced yes)
 		(property "Reference" "U1"
-			(at 39.37 20.32 0)
+			(at 43.18 96.52 0)
 			(effects
 				(font
@@
 		)
 		(property "Value" "TPS22917DBVR"
-			(at 39.37 22.86 0)
+			(at 43.18 99.06 0)
 			(effects
 				(font
@@
 		)
 		(property "Footprint" "parts:SOT95P280X145-6N"
-			(at 39.37 35.56 0)
+			(at 43.18 111.76 0)
 			(effects
 				(font
@@
 		)
 		(property "Datasheet" ""
-			(at 39.37 35.56 0)
+			(at 43.18 111.76 0)
 			(effects
 				(font
@@
 		)
 		(property "Description" ""
-			(at 39.37 35.56 0)
+			(at 43.18 111.76 0)
 			(effects
 				(font
@@
 		)
 		(property "PARTREV" "B"
-			(at 39.37 35.56 0)
+			(at 43.18 111.76 0)
 			(effects
 				(font
@@
 		)
 		(property "STANDARD" "IPC 7351B"
-			(at 39.37 35.56 0)
+			(at 43.18 111.76 0)
 			(effects
 				(font
@@
 		)
 		(property "MAXIMUM_PACKAGE_HEIGHT" "1.45mm"
-			(at 39.37 35.56 0)
+			(at 43.18 111.76 0)
 			(effects
 				(font
@@
 		)
 		(property "MANUFACTURER" "Texas Instruments"
-			(at 39.37 35.56 0)
-			(effects
-				(font
+			(at 43.18 111.76 0)
+			(effects
+				(font

Commit message: changed parts to 400MHz version
Parts:
- added C29: ~, parts:C0603, symbol MB1389-altium-import:U_STM32_microcontroller_RF_1_Capacitor
- added C32: ~, parts:C0402, symbol MB1389-altium-import:U_STM32_microcontroller_RF_3_Capacitor
Connections:
- net GND: now also C29.1, C32.2
- net VGPS: now also C29.2, C32.1

Commit message: bom changes
Parts:
- U1: MANUFACTURER Texas Instruments -> (none); MAXIMUM_PACKAGE_HEIGHT 1.45mm -> (none); PARTREV B -> (none); STANDARD IPC 7351B -> (none)
Changed lines of the file:
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@@
 			)
 		)
-		(property "Datasheet" "SAM-M10Q-00B"
+		(property "Datasheet" "https://www.digikey.com/en/products/detail/u-blox/SAM-M10Q-00B/16672678"
 			(at 138.43 78.74 0)
 			(effects
@@
 			)
 		)
-		(property "Datasheet" ""
+		(property "Datasheet" "https://www.digikey.com/en/products/detail/texas-instruments/TPS22917DBVR/8539916"
 			(at 43.18 111.76 0)
 			(effects
@@
 				(hide yes)
 			)
-		)
-		(property "PARTREV" "B"
-			(at 43.18 111.76 0)
-			(effects
-				(font
-					(size 1.27 1.27)
-				)
-				(justify bottom)
-				(hide yes)
-			)
-		)
-		(property "STANDARD" "IPC 7351B"
-			(at 43.18 111.76 0)
-			(effects
-				(font
-					(size 1.27 1.27)
-				)
-				(justify bottom)
-				(hide yes)
-			)
-		)
-		(property "MAXIMUM_PACKAGE_HEIGHT" "1.45mm"
-			(at 43.18 111.76 0)
-			(effects
-				(font
-					(size 1.27 1.27)
-				)
-				(justify bottom)
-				(hide yes)
-			)
-		)
-		(property "MANUFACTURER" "Texas Instruments"
-			(at 43.18 111.76 0)
-			(effects
-				(font
-					(size 1.27 1.27)
-				)
-				(justify bottom)
-				(hide yes)
-			)

Commit message: finished bom
Parts:
- C29: value ~ -> 4.7uF; ALTIUM_VALUE 4.7uF -> (none); MANUFACTURER_PART_NUMBER CC0603KRX5R7BB475 -> (none)
- C32: value ~ -> 100nF; ALTIUM_VALUE 100nF -> (none); MANUFACTURER_PART_NUMBER CC0402KRX7R7BB104 -> (none)
