File: radioboard_dev/radioboard_dev.kicad_pcb (KiCad board)
At the start: 4 copper layers, 32.5 x 148.2 mm, 103 parts, among them J1 Conn_01x02, J2 Conn_01x02, J3 Conn_01x04, J4 Conn_01x04, J5 Conn_01x04, J6 Conn_01x04, J9 Conn_01x04, U1 TPS22917DBVR, U10 STM32WL55CCUx, U11 MAX17048G_T10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

Commit message: finished bom
Parts:
- C1, C26, C29, C3, C35, C4: value ~ -> 4.7uF
- C10, C18, C23, C28, C32, C37, C67, C77, C9: value ~ -> 100nF
- C11, C14: value 15 pF -> 15pF
- C12, C13: value Capacitor -> 68pF
- C15: value 4.3 pF -> 4.3pF
- C16: value 3.6 pF -> 3.6pF
- C20: value ~ -> 3.6pF
- C27: value Capacitor -> 220nF
- C30, C38: value ~ -> 6.8pF
- C31: value Capacitor -> 10pF
- C43, C44: value ~ -> 5.1pF
- C7, C8: value Capacitor -> 5.6pF
- C71, C72, C73: value ~ -> 1nF
- C74: value ~ -> 47nF
- C76: value ~ -> 68pF
- C79: value ~ -> 47pF
- C85: value ~ -> 470nF
- L13: value ~ -> 15µH
- R2: value Resistor -> 220R
- R26, R4: value ~ -> 10k
- R27, R28, R29: value ~ -> 220R
- R3, R35: value ~ -> 270R
- R34: value ~ -> 360R
- turned R27 to 180 degrees
- turned R28 to 180 degrees
- turned R29 to 0 degrees
Connections:
- R27 pad 1: /microcontroller_RF/FE_CTRL1 -> Net-(U8-V1)
- R27 pad 2: Net-(U8-V1) -> /microcontroller_RF/FE_CTRL1
- R28 pad 1: /microcontroller_RF/FE_CTRL2 -> Net-(U8-V2)
- R28 pad 2: Net-(U8-V2) -> /microcontroller_RF/FE_CTRL2
- R29 pad 1: Net-(U8-VDD) -> /microcontroller_RF/FE_CTRL3
- R29 pad 2: /microcontroller_RF/FE_CTRL3 -> Net-(U8-VDD)
- U12 pad : GND -> (no net)
