File: radioboard_dev/STM32_microcontroller_IOs.kicad_sch (KiCad schematic)
At the start: 20 parts, among them U10 STM32WL55CCUx

Commit message: finished bom
Parts:
- C10, C23, C28, C67: value ~ -> 100nF; ALTIUM_VALUE 100nF -> (none); MANUFACTURER_PART_NUMBER CC0402KRX7R7BB104 -> (none)
- C18: value ~ -> 100nF; footprint Capacitor_SMD:C_0402_1005Metric -> parts:C0402; ALTIUM_VALUE 100nF -> (none); MANUFACTURER_PART_NUMBER CC0402KRX7R7BB104 -> (none)
- C26: value ~ -> 4.7uF; ALTIUM_VALUE 4.7uF -> (none); MANUFACTURER_PART_NUMBER CC0603KRX5R7BB475 -> (none)
- C43, C44: value ~ -> 5.1pF; ALTIUM_VALUE 5.1pF -> (none); COMPONENTLINK1DESCRIPTION Datasheet -> (none); COMPONENTLINK1URL http://tunmcdsvn.tun.st.com/Component_Datasheet_Library/Tru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 -> (none); ECCN_EU NEC -> (none); ECCN_US EAR99 -> (none); INTERNAL_PART_NUMBER MCD-00003 -> (none); MANUFACTURER YAGEO -> (none); MANUFACTURER_PART_NUMBER CC0402CRNPO9BN5R1 -> (none); PACKAGE C0402 -> (none); PART_TYPE Capacitor -> (none); PROVIDED_BY SUBCO -> (none); STATUS Released -> (none)
- L1: ALTIUM_VALUE 600R@100MHz -> (none); MANUFACTURER_PART_NUMBER FCM1608KF-601T03 -> (none)
- R26, R4: value ~ -> 10k; ALTIUM_VALUE 10K -> (none); COMPONENTLINK1DESCRIPTION Datasheet -> (none); COMPONENTLINK1URL http://tunmcdsvn.tun.st.com/Component_Datasheet_Library/Tru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 -> (none); ECCN_EU NEC -> (none); ECCN_US EAR99 -> (none); INTERNAL_PART_NUMBER MCD-00220 -> (none); MANUFACTURER YAGEO -> (none); MANUFACTURER_PART_NUMBER RC0603FR-0710KL -> (none); PACKAGE R0603 -> (none); PART_TYPE Resistor -> (none); PROVIDED_BY SUBCO -> (none); STATUS Released -> (none)
- R34: value ~ -> 360R; ALTIUM_VALUE 360R -> (none); COMPONENTLINK1DESCRIPTION Datasheet -> (none); COMPONENTLINK1URL http://tunmcdsvn.tun.st.com/Component_Datasheet_Library/Tru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 -> (none); ECCN_EU NEC -> (none); ECCN_US EAR99 -> (none); INTERNAL_PART_NUMBER MCD-00461 -> (none); MANUFACTURER YAGEO -> (none); MANUFACTURER_PART_NUMBER RC0402FR-07360RL -> (none); PACKAGE R0402 -> (none); PART_TYPE Resistor -> (none); PROVIDED_BY SUBCO -> (none); STATUS Released -> (none)
- R35: value ~ -> 270R; footprint R0402 -> parts:R0402; ALTIUM_VALUE 270R -> (none); COMPONENTLINK1DESCRIPTION Datasheet -> (none); COMPONENTLINK1URL http://tunmcdsvn.tun.st.com/Component_Datasheet_Library/Tru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 -> (none); ECCN_EU NEC -> (none); ECCN_US EAR99 -> (none); INTERNAL_PART_NUMBER MCD-00441 -> (none); MANUFACTURER YAGEO -> (none); MANUFACTURER_PART_NUMBER RC0402FR-07270RL -> (none); PACKAGE R0402 -> (none); PART_TYPE Resistor -> (none); PROVIDED_BY SUBCO -> (none); STATUS Released -> (none)

Commit message: removed HW20
Parts:
- removed HW20: ~, symbol MB1389-altium-import:U_STM32_microcontroller_IOs_0_Shunt Black 2.54mm
